Commit message: migrate to x64 system for cartographer bug

File: derobotee/urdf/diff_wheeled_robot.xacro (robot description, xacro)
@@ -82,5 +82,5 @@
       <geometry>
           <!--cylinder length="${base_height}" radius="${base_radius}" /-->
-          <box size="0.5 0.42 0.05" />
+          <box size="0.8 0.62 0.05" />
       </geometry>
       <material name="White" />
@@ -123,5 +123,5 @@
       <parent link="base_link"/>
       <child link="caster_front_link"/>
-      <origin xyz="0.238 0.0 0" rpy="${-M_PI/2} 0 0"/>
+      <origin xyz="0.538 0.0 0" rpy="${-M_PI/2} 0 0"/>
     </joint>
   <gazebo reference="caster_front_link">
@@ -133,4 +133,18 @@
   <!-- SENSORS -->
   <!-- hokuyo -->
+  <link name="imu_link">
+   <visual>
+     <origin xyz="0 0 0"/>
+     <geometry>
+       <box size="0.06 0.04 0.02" />
+     </geometry>
+     <material name="orange" />
+   </visual>
+  </link>
+  <joint name="imu_link_joint" type="fixed">
+i   <parent link="base_link" />
+    <child link="imu_link" />
+    <origin xyz="0 0 0.3" rpy="0.1  0.1  0"/>
+  </joint>
   <link name="hokuyo_link">
     <visual>
@@ -143,5 +157,5 @@
   </link>
   <joint name="hokuyo_joint" type="fixed">
-    <origin xyz="0.43805 0 ${base_height+hokuyo_size/4}" rpy="0 0 ${-M_PI}" />
+    <origin xyz="0.52638 0 0.20" rpy="0 0.01 0" />
     <parent link="base_link"/>
     <child link="hokuyo_link" />

File: derobotee/urdf/wheel.urdf.xacro (robot description, xacro)
@@ -3,8 +3,8 @@
   <!-- Wheels -->
   <property name="wheel_radius" value="0.065" />
-  <property name="wheel_height" value="0.035" />
+  <property name="wheel_height" value="0.042" />
   <property name="wheel_mass" value="2.5" /> <!-- in kg-->
   <property name="base_x_origin_to_wheel_origin" value="0" />
-  <property name="base_y_origin_to_wheel_origin" value="0.132" />
+  <property name="base_y_origin_to_wheel_origin" value="0.264" />
   <property name="base_z_origin_to_wheel_origin" value="0.0" />
   <macro name="cylinder_inertia" params="m r h">
@@ -47,5 +47,5 @@
       <child link="${fb}_${lr}_wheel"/>
       <origin xyz="${translateX * base_x_origin_to_wheel_origin} ${translateY * base_y_origin_to_wheel_origin} ${base_z_origin_to_wheel_origin}" rpy="0 0 0" />
-      <axis xyz="0 1 0" rpy="0  0" />
+      <axis xyz="0 1 0" rpy="0 0 0" />
       <limit effort="100" velocity="100"/>
       <joint_properties damping="0.0" friction="0.0"/>

Commit message: build map successfully

File: derobotee/urdf/diff_wheeled_robot.xacro (robot description, xacro)
@@ -37,5 +37,5 @@
 -->
   <!-- Hokuyo Laser scanner -->
-  <property name="hokuyo_size" value="0.15" />
+  <property name="sick_size" value="0.15" />
   <!-- Macro for calculating inertia of cylinder -->
   <macro name="cylinder_inertia" params="m r h">
@@ -65,5 +65,5 @@
   </gazebo>
   <joint name="base_footprint_joint" type="fixed">
-    <origin xyz="0 0 ${wheel_radius - base_z_origin_to_wheel_origin}" rpy="0 0 0" />
+    <origin xyz="0 0 ${wheel_radius - base_z_origin_to_wheel_origin}" rpy="0 0.01 0" />
     <parent link="base_footprint"/>
     <child link="base_link" />
@@ -137,5 +137,5 @@
      <origin xyz="0 0 0"/>
      <geometry>
-       <box size="0.06 0.04 0.02" />
+       <box size="0.035 0.035 0.02" />
      </geometry>
      <material name="orange" />
@@ -145,25 +145,25 @@
 i   <parent link="base_link" />
     <child link="imu_link" />
-    <origin xyz="0 0 0.3" rpy="0.1  0.1  0"/>
+    <origin xyz="0.404 0.2395 0.008" rpy="0  0  0"/>
   </joint>
-  <link name="hokuyo_link">
+  <link name="laser">
     <visual>
       <origin xyz="0 0 0" rpy="0 0 0" />
       <geometry>
-        <box size="${hokuyo_size} ${hokuyo_size} ${hokuyo_size}"/>
+        <box size="${sick_size} ${sick_size} ${sick_size}"/>
       </geometry>
       <material name="Blue" />
     </visual>
   </link>
-  <joint name="hokuyo_joint" type="fixed">
-    <origin xyz="0.52638 0 0.20" rpy="0 0.01 0" />
+  <joint name="sick_joint" type="fixed">
+    <origin xyz="0.52638 0 0.20" rpy="0 0 0" />
     <parent link="base_link"/>
-    <child link="hokuyo_link" />
+    <child link="laser" />
   </joint>
-  <gazebo reference="hokuyo_link">
+  <gazebo reference="laser">
     <material>Gazebo/Blue</material>
     <turnGravityOff>false</turnGravityOff>
     <sensor type="ray" name="head_hokuyo_sensor">
-      <pose>${hokuyo_size/2} 0 0 0 0 0</pose>
+      <pose>${sick_size/2} 0 0 0 0 0</pose>
       <visualize>false</visualize>
       <update_rate>40</update_rate>
@@ -185,5 +185,5 @@
       <plugin name="gazebo_ros_head_hokuyo_controller" filename="libgazebo_ros_laser.so">
         <topicName>/scan</topicName>
-        <frameName>hokuyo_link</frameName>
+        <frameName>laser</frameName>
       </plugin>
     </sensor>
